File: Base_Portenta_Stack/BASE_Portenta_H7_stack.kicad_pcb (KiCad board)
At the start: 2 copper layers, 82.1 x 26.7 mm, 22 parts, among them J4 PinHeader_1x04_P2.00mm_Vertic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, U1 ABX00042

Commit message: Log
Parts:
- removed the REF** at (183.0, 95.3)
- added REF**: C_0805_2012Metric, Capacitor_SMD:C_0805_2012Metric, B.Cu at (169.7, 99.3)
- added REF**: JST_PH_S6B-PH-SM4-TB_1x06-1MP_P2.00mm_Horizontal, Connector_JST:JST_PH_S6B-PH-SM4-TB_1x06-1MP_P2.00mm_Horizontal, F.Cu at (99.9, 88.9)
- added REF**: PinHeader_1x02_P2.54mm_Vertical, Connector_PinHeader_2.54mm:PinHeader_1x02_P2.54mm_Vertical, F.Cu at (182.4, 84.8)
- added REF**: PinHeader_1x02_P2.54mm_Vertical, Connector_PinHeader_2.54mm:PinHeader_1x02_P2.54mm_Vertical, F.Cu at (182.6, 102.6)
- added REF**: C_0805_2012Metric, Capacitor_SMD:C_0805_2012Metric, B.Cu at (171.9, 101.8)
- CAN FD: renamed from REF**; value PinHeader_1x04_P2.54mm_Vertical -> PinHeader_1x03_P2.54mm_Vertical; footprint Connector_PinHeader_2.54mm:PinHeader_1x04_P2.54mm_Vertical -> Connector_PinHeader_2.54mm:PinHeader_1x03_P2.54mm_Vertical
- moved CAN FD 87.4 mm to (97.1, 99.8)
- moved REF** 4.92 mm to (172.1, 93.8)
- moved REF** 1.42 mm to (170.0, 93.8)
- moved REF** 1.26 mm to (172.3, 89.0)
- moved REF** 1.26 mm to (172.3, 87.6)
- moved REF** 1.26 mm to (172.3, 86.1)
- moved REF** 1.25 mm to (166.6, 93.8)
- moved REF** 0.79 mm to (176.4, 94.1)
- moved REF** 0.66 mm to (174.4, 82.7)
- moved REF** 0.66 mm to (177.7, 82.7)
- moved REF** 0.24 mm to (175.5, 104.0)
Routing:
- added copper zone on B.Cu, net VIN
Other:
- board size 82.1 x 26.7 mm -> 89.5 x 26.7 mm
- board text removed: "12V"
- board text removed: "CAN"
- board text removed: "HALL"
